File: hardware/ClassicsController.kicad_sch (KiCad schematic)
At the start: 6 parts

Commit message: Schematic about half done
- Most main ICs on schematic
- Some bus connections made (About 50%)
- All logic ICs and 6802 still need decoupling
- Design validation still needs to happen
- Some basic/initial floorplanning done on PCB
- All and all, a decent start
Parts:
- removed U?: MC68A02, Package_DIP:DIP-40_W15.24mm, symbol CPU_NXP_6800:MC68A02
- added C1, C15, C16, C2, C3: C, Capacitor_SMD:C_0805_2012Metric, symbol Device:C
- added C10, C11, C12, C4, C5, C6, C7, C8, C9: 0.1uF, Capacitor_SMD:C_0805_2012Metric, symbol Device:C
- added C13, C14: 1uF, Capacitor_SMD:C_0805_2012Metric, symbol Device:C
- added C17, C18: 27pF, Capacitor_SMD:C_0805_2012Metric, symbol Device:C
- added C19, C20: 27pF, symbol Device:C
- added D1: D_Schottky, Diode_SMD:D_1206_3216Metric, symbol Device:D_Schottky
- added FB1: FerriteBead, Inductor_SMD:L_0603_1608Metric_Pad1.05x0.95mm_HandSolder, symbol Device:FerriteBead_Small
- added JP1: Jumper_2_Open, Connector_PinHeader_2.54mm:PinHeader_1x02_P2.54mm_Vertical, symbol Jumper:Jumper_2_Open
- added JP2: SolderJumper_2_Open, Jumper:SolderJumper-2_P1.3mm_Open_TrianglePad1.0x1.5mm, symbol Jumper:SolderJumper_2_Open
- added R1: DNP, Resistor_SMD:R_0603_1608Metric, symbol Device:R
- added R2: 1k, Resistor_SMD:R_0603_1608Metric, symbol Device:R
- added R3: 3.3k, Resistor_SMD:R_0603_1608Metric, symbol Device:R
- added R4: 330, Resistor_SMD:R_0603_1608Metric, symbol Device:R
- added R5, R6: 27.4, Resistor_SMD:R_0603_1608Metric, symbol Device:R
- added R7: 1k, symbol Device:R
- added SW1, SW2: SW_SPST, Button_Switch_SMD:SW_SPST_CK_RS282G05A3, symbol Switch:SW_SPST
- added TP1, TP2, TP3, TP4: TestPoint, symbol Connector:TestPoint
- added U1: MC6802, Package_DIP:DIP-40_W15.24mm, symbol CPU_NXP_6800:MC6802
- added U10, U9: SN74CBT16245CDL, Package_SO:SSOP-48_7.5x15.9mm_P0.635mm, symbol 74xx:SN74CBT16245CDL
- added U3: W25Q128JVS, Package_SO:SOIC-8_5.23x5.23mm_P1.27mm, symbol Memory_Flash:W25Q128JVS
- added U4: TXB0108PWR, Package_SO:TSSOP-20_4.4x6.5mm_P0.65mm, symbol Logic_LevelTranslator:TXB0108PWR
- added U7, U8: SN74CBT16233DGGR, Package_SO:TSSOP-56_6.1x14mm_P0.5mm, symbol SN74CBT16233DGGR:SN74CBT16233DGGR
- added Y1: 3.58Mhz, Crystal:Crystal_HC52-U_Vertical, symbol Device:Crystal
- added Y2: Crystal, symbol Device:Crystal
- J2: renamed from J?; footprint (none) -> Connector_IDC:IDC-Header_2x20_P2.54mm_Vertical
- gave numbers to parts that had none: 4
Connections:
- net VBUS: now reaches J1.1 (VBUS)
- net VBUS: now also D1.2 (A)
- net USB_DM: now reaches J1.2 (D-)
- net USB_DM: now also R6.1
- net USB_DP: now reaches J1.3 (D+)
- net USB_DP: now also R5.1
- net GND: now reaches J1.4 (GND)
- net GND: now also U2.57 (GND), U5.11 (A0), U5.12 (A1), U5.13 (A2), U5.29 (EP), U5.6 (VSS), U6.12 (A1), U6.13 (A2), U6.29 (EP), U6.6 (VSS), C1.2, C10.2, C11.2, C12.2, C13.2, C14.2, C15.2, C16.2, C17.1, C18.1, C19.1, C2.2, C20.1, C3.2, C4.2, C5.2, C6.2, C7.2, C8.2, C9.2, FB1.1, R2.2, R4.1, U1.1 (VSS), U1.21 (VSS), U3.4 (GND), U4.11 (GND)
- net at J1.5 (Shield): now also FB1.2
- net RP_SPI_MISO_H: now reaches U5.10 (SO)
- net RP_SPI_MISO_H: now also U6.10 (SO), TP4.1, U4.17 (B3)
- net PICO_D0: now reaches U5.17 (GPA0)
- net PICO_D0: now also U7.55 (1B2)
- net PICO_D1: now reaches U5.18 (GPA1)
- net PICO_D1: now also U7.3 (2B2)
- net PICO_D2: now reaches U5.19 (GPA2)
- net PICO_D2: now also U7.52 (3B2)
- net PICO_D3: now reaches U5.20 (GPA3)
- net PICO_D3: now also U7.6 (4B2)
- net PICO_D4: now reaches U5.21 (GPA4)
- net PICO_D4: now also U7.49 (5B2)
- net PICO_D5: now reaches U5.22 (GPA5)
- net PICO_D5: now also U7.9 (6B2)
- net PICO_D6: now reaches U5.23 (GPA6)
- net PICO_D6: now also U7.46 (7B2)
- net PICO_D7: now reaches U5.24 (GPA7)
- net PICO_D7: now also U7.12 (8B2)
- net +5V: now reaches U5.5 (VDD)
- net +5V: now also U6.11 (A0), U6.5 (VDD), C16.1, C2.1, C3.1, JP1.2 (B), JP2.2 (B), U4.19 (VCCB)
- net RP_SPI_CS_H: now reaches U5.7 (~{CS})
- net RP_SPI_CS_H: now also U6.7 (~{CS}), TP1.1, U4.16 (B4)
- net RP_SPI_CLK_H: now reaches U5.8 (SCK)
- net RP_SPI_CLK_H: now also U6.8 (SCK), TP2.1, U4.20 (B1)
- net RP_SPI_MOSI_H: now reaches U5.9 (SI)
- net RP_SPI_MOSI_H: now also U6.9 (SI), TP3.1, U4.18 (B2)
- net +3.3V: now reaches U2.1 (IOVDD), U2.10 (IOVDD), U2.22 (IOVDD), U2.33 (IOVDD), U2.42 (IOVDD), U2.49 (IOVDD)
- net +3.3V: now also U2.43 (ADC_AVDD), U2.44 (VREG_IN), U2.48 (USB_VDD), C1.1, C10.1, C11.1, C12.1, C14.1, C15.1, C6.1, C7.1, C8.1, C9.1, R1.1, R3.1, U3.8 (VCC), U4.2 (VCCA)
- net at U2.20 (XIN): now also C19.2, Y2.1
- net at U2.21 (XOUT): now also R7.2
- net +1V1: now reaches U2.23 (DVDD), U2.50 (DVDD)
- net +1V1: now also U2.45 (VREG_VOUT), C13.1, C4.1, C5.1
- net at U2.26 (RUN): now also R3.2, SW2.2 (B)
- net RP_SPI_CLK_L: now reaches U2.4 (GPIO2)
- net RP_SPI_CLK_L: now also U4.1 (A1)
- net at U2.46 (USB_DM): now also R6.2
- net at U2.47 (USB_DP): now also R5.2
- net RP_SPI_MOSI_L: now reaches U2.5 (GPIO3)
- net RP_SPI_MOSI_L: now also U4.3 (A2)
- net QSPI_SD3: now reaches U2.51 (QSPI_SD3)
- net QSPI_SD3: now also U3.7 (IO3)
- net QSPI_SCLK: now reaches U2.52 (QSPI_SCLK)
- net QSPI_SCLK: now also U3.6 (CLK)
- net QSPI_SD0: now reaches U2.53 (QSPI_SD0)
- net QSPI_SD0: now also U3.5 (DI(IO0))
- net QSPI_SD2: now reaches U2.54 (QSPI_SD2)
- net QSPI_SD2: now also U3.3 (IO2)
- net QSPI_SD1: now reaches U2.55 (QSPI_SD1)
- net QSPI_SD1: now also U3.2 (DO(IO1))
- net QSPI_SS: now reaches U2.56 (QSPI_SS)
- net QSPI_SS: now also R1.2, SW1.2 (B), U3.1 (~{CS})
- net RP_SPI_MISO_L: now reaches U2.6 (GPIO4)
- net RP_SPI_MISO_L: now also U4.4 (A3)
- net RP_SPI_CS_L: now reaches U2.7 (GPIO5)
- net RP_SPI_CS_L: now also U4.5 (A4)
- net PICO_A12: now reaches U6.1 (GPB4)
- net PICO_A12: now also U8.35 (13B2)
- net PICO_A0: now reaches U6.17 (GPA0)
- net PICO_A0: now also U8.55 (1B2)
- net PICO_A1: now reaches U6.18 (GPA1)
- net PICO_A1: now also U8.3 (2B2)
- net PICO_A2: now reaches U6.19 (GPA2)
- net PICO_A2: now also U8.52 (3B2)
- net PICO_A13: now reaches U6.2 (GPB5)
- net PICO_A13: now also U8.23 (14B2)
- net PICO_A3: now reaches U6.20 (GPA3)
- net PICO_A3: now also U8.6 (4B2)
- net PICO_A4: now reaches U6.21 (GPA4)
- net PICO_A4: now also U8.49 (5B2)
- net PICO_A5: now reaches U6.22 (GPA5)
- net PICO_A5: now also U8.9 (6B2)
- net PICO_A6: now reaches U6.23 (GPA6)
- net PICO_A6: now also U8.46 (7B2)
- net PICO_A7: now reaches U6.24 (GPA7)
- net PICO_A7: now also U8.12 (8B2)
- net PICO_A8: now reaches U6.25 (GPB0)
- net PICO_A8: now also U8.41 (9B2)
- net PICO_A9: now reaches U6.26 (GPB1)
- net PICO_A9: now also U8.17 (10B2)
- net PICO_A10: now reaches U6.27 (GPB2)
- net PICO_A10: now also U8.38 (11B2)
- net PICO_A11: now reaches U6.28 (GPB3)
- net PICO_A11: now also U8.20 (12B2)
- net PICO_A14: now reaches U6.3 (GPB6)
- net PICO_A14: now also U8.32 (15B2)
- net PICO_A15: now reaches U6.4 (GPB7)
- net PICO_A15: now also U8.26 (16B2)
- new net: C17.2, U1.38 (XTAL), Y1.1
- new net: C18.2, U1.39 (EXTAL), Y1.2
- new net: R4.2, SW2.1 (A)
- new net: R2.1, SW1.1 (A)
- new net: U9.10 (GND), U9.15 (GND), U9.21 (GND), U9.28 (GND), U9.34 (GND), U9.39 (GND), U9.4 (GND), U9.45 (GND)
- new net: U9.18 (VCC), U9.31 (VCC), U9.42 (VCC), U9.7 (VCC)
- new net: D1.1 (K), JP1.1 (A), JP2.1 (A)
- new net: C20.2, R7.1, Y2.2
- new net: U10.10 (GND), U10.15 (GND), U10.21 (GND), U10.28 (GND), U10.34 (GND), U10.39 (GND), U10.4 (GND), U10.45 (GND)
- new net: U10.18 (VCC), U10.31 (VCC), U10.42 (VCC), U10.7 (VCC)
- new net 6802_A0: U1.9 (A0), U8.56 (1B1)
- new net 6802_A1: U1.10 (A1), U8.2 (2B1)
- new net 6802_A10: U1.19 (A10), U8.39 (11B1)
- new net 6802_A11: U1.20 (A11), U8.19 (12B1)
- new net 6802_A12: U1.22 (A12), U8.36 (13B1)
- new net 6802_A13: U1.23 (A13), U8.22 (14B1)
- new net 6802_A14: U1.24 (A14), U8.33 (15B1)
- new net 6802_A15: U1.25 (A15), U8.25 (16B1)
- new net 6802_A2: U1.11 (A2), U8.53 (3B1)
- new net 6802_A3: U1.12 (A3), U8.5 (4B1)
- new net 6802_A4: U1.13 (A4), U8.50 (5B1)
- new net 6802_A5: U1.14 (A5), U8.8 (6B1)
- new net 6802_A6: U1.15 (A6), U8.47 (7B1)
- new net 6802_A7: U1.16 (A7), U8.11 (8B1)
- new net 6802_A8: U1.17 (A8), U8.42 (9B1)
- new net 6802_A9: U1.18 (A9), U8.16 (10B1)
- new net 6802_D0: U1.33 (D0), U7.56 (1B1)
- new net 6802_D1: U1.32 (D1), U7.2 (2B1)
- new net 6802_D2: U1.31 (D2), U7.53 (3B1)
- new net 6802_D3: U1.30 (D3), U7.5 (4B1)
- new net 6802_D4: U1.29 (D4), U7.50 (5B1)
- new net 6802_D5: U1.28 (D5), U7.8 (6B1)
- new net 6802_D6: U1.27 (D6), U7.47 (7B1)
- new net 6802_D7: U1.26 (D7), U7.11 (8B1)
- new net SW_A0: U10.2 (B0), U8.1 (1A)
- new net SW_A1: U10.3 (B1), U8.54 (2A)
- new net SW_A10: U10.16 (B10), U8.18 (11A)
- new net SW_A11: U10.17 (B11), U8.37 (12A)
- new net SW_A12: U10.19 (B12), U8.21 (13A)
- new net SW_A13: U10.20 (B13), U8.34 (14A)
- new net SW_A14: U10.22 (B14), U8.24 (15A)
- new net SW_A15: U10.23 (B15), U8.31 (16A)
- new net SW_A2: U10.5 (B2), U8.4 (3A)
- new net SW_A3: U10.6 (B3), U8.51 (4A)
- new net SW_A4: U10.8 (B4), U8.7 (5A)
- new net SW_A5: U10.9 (B5), U8.48 (6A)
- new net SW_A6: U10.11 (B6), U8.10 (7A)
- new net SW_A7: U10.12 (B7), U8.45 (8A)
- new net SW_A8: U10.13 (B8), U8.15 (9A)
- new net SW_A9: U10.14 (B9), U8.40 (10A)
- no-connect marks 0 -> 2
Other:
- note added: "Pico Flash Memory"
- note added: "TODO: -Finish connecting busses -Support circuitry for logic ICs -Thorough decoupling -Connect J2 as if it were 6802 -Cleanup/improve floorplanning"
- note added: "USB Input"
- moved on the sheet: J1, J2, U2, U5, U6

Commit message: Improve Bussing in Schematic
- Most bussing is done.
- Improved the symbol for SN74CBT16233DGGR to accomodate all the busses.
Connections:
- net GND: now also U7.13 (GND), U7.44 (GND), U8.13 (GND), U8.44 (GND)
- net 6802_R/~{W}: now reaches U1.34 (R/~{W})
- net 6802_R/~{W}: now also U7.42 (9B1)
- net 6802_Phi2: now reaches U1.37 (E)
- net 6802_Phi2: now also U7.16 (10B1)
- net ~{6802_IRQ}: now reaches U1.4 (~{IRQ})
- net ~{6802_IRQ}: now also U7.19 (12B1)
- net ~{6802_RESET}: now reaches U1.40 (~{RESET})
- net ~{6802_RESET}: now also U7.22 (14B1)
- net 6802_VMA: now reaches U1.5 (VMA)
- net 6802_VMA: now also U7.39 (11B1)
- net ~{6802_NMI}: now reaches U1.6 (~{NMI})
- net ~{6802_NMI}: now also U7.36 (13B1)
- net SW_D0: now reaches U7.1 (1A)
- net SW_D0: now also U9.2 (B0)
- net SW_D6: now reaches U7.10 (7A)
- net SW_D6: now also U9.11 (B6)
- net VCC: now reaches U7.14 (VCC)
- net VCC: now also U7.43 (VCC), U8.14 (VCC), U8.43 (VCC)
- net SW_R/~{W}: now reaches U7.15 (9A)
- net SW_R/~{W}: now also U9.13 (B8)
- net PICO_Phi2: now reaches U7.17 (10B2)
- net PICO_Phi2: now also U5.26 (GPB1)
- net SW_VMA: now reaches U7.18 (11A)
- net SW_VMA: now also U9.16 (B10)
- net ~{PICO_IRQ}: now reaches U7.20 (12B2)
- net ~{PICO_IRQ}: now also U5.28 (GPB3)
- net ~{SW_NMI}: now reaches U7.21 (13A)
- net ~{SW_NMI}: now also U9.19 (B12)
- net ~{PICO_RESET}: now reaches U7.23 (14B2)
- net ~{PICO_RESET}: now also U5.2 (GPB5)
- net ~{SW_RESET}: now reaches U7.34 (14A)
- net ~{SW_RESET}: now also U9.20 (B13)
- net ~{PICO_NMI}: now reaches U7.35 (13B2)
- net ~{PICO_NMI}: now also U5.1 (GPB4)
- net ~{SW_IRQ}: now reaches U7.37 (12A)
- net ~{SW_IRQ}: now also U9.17 (B11)
- net PICO_VMA: now reaches U7.38 (11B2)
- net PICO_VMA: now also U5.27 (GPB2)
- net SW_D2: now reaches U7.4 (3A)
- net SW_D2: now also U9.5 (B2)
- net SW_Phi2: now reaches U7.40 (10A)
- net SW_Phi2: now also U9.14 (B9)
- net PICO_R/~{W}: now reaches U7.41 (9B2)
- net PICO_R/~{W}: now also U5.25 (GPB0)
- net SW_D7: now reaches U7.45 (8A)
- net SW_D7: now also U9.12 (B7)
- net SW_D5: now reaches U7.48 (6A)
- net SW_D5: now also U9.9 (B5)
- net SW_D3: now reaches U7.51 (4A)
- net SW_D3: now also U9.6 (B3)
- net SW_D1: now reaches U7.54 (2A)
- net SW_D1: now also U9.3 (B1)
- net SW_D4: now reaches U7.7 (5A)
- net SW_D4: now also U9.8 (B4)
